Commit message: General update, rework of file-structure and content

File: urdf/robot_srdf.xacro (robot description, xacro)
@@ -1,4 +1,5 @@
 <?xml version="1.0" ?>
-<robot name="robot_scene" xmlns:xacro="http://ros.org/wiki/xacro">
+<robot name="robot" xmlns:xacro="http://ros.org/wiki/xacro">
+  <xacro:macro name="robot" params="robot_prefix robot_type">
   <!-- Xacro Parameters -->
   <xacro:arg name="robot_prefix"  default=""/>
@@ -10,4 +11,5 @@
     <!-- The Yaskawa-Robot-SRDF xacro must be included with passing parameters -->
     <xacro:include filename="$(find robot_support)/urdf/robots/gp400/gp400_srdf.xacro"/>
+    <!-- The xacro must be included with passing parameters -->
     <!-- "robot_prefix" describes the naming of the robot -->
     <xacro:robot_gp400 robot_prefix = "$(arg robot_prefix)"/>
@@ -17,6 +19,8 @@
     <!-- The ABB-Robot-URDF xacro must be included with passing parameters -->
     <xacro:include filename="$(find robot_support)/urdf/robots/irb6660/irb6660_srdf.xacro"/>
+    <!-- The xacro must be included with passing parameters -->
     <!-- "prefix" describes the naming of the robot -->
     <xacro:robot_irb6660 robot_prefix = "$(arg robot_prefix)"/>
   </xacro:if>
+  </xacro:macro>
 </robot>
