Commit message: Fixed package naming reference

File: urdf/environment/toolstand/toolstand_macro.xacro (robot description, xacro)
@@ -17,5 +17,5 @@
                 <origin xyz="0.0 0.0 1.17" rpy="${radians(-90)} 0 0"/>
                 <geometry>
-                    <mesh filename="package://robotics_support/environment/toolstand/meshes/visual/toolstand.stl"/>
+                    <mesh filename="package://robot_support/environment/toolstand/meshes/visual/toolstand.stl"/>
                 </geometry>
                 <material name="${prefix}_dark_grey"/>
@@ -25,5 +25,5 @@
                 <geometry>
                     <!-- using "visual" as collision mesh, to allow robot interaction -->
-                    <mesh filename="package://robotics_support/environment/toolstand/meshes/visual/toolstand.stl"/>
+                    <mesh filename="package://robot_support/environment/toolstand/meshes/visual/toolstand.stl"/>
                 </geometry>
             </collision>
