Commit message: Changed prefix addition to accomodate dual-robot scene

File: urdf/robots/gp400/gp400_srdf.xacro (robot description, xacro)
@@ -14,89 +14,89 @@
     <!--SUBGROUPS: Groups can also be formed by referencing to already defined group names-->
     <!-- Robot Manipulator -->
-    <group name="$(arg robot_prefix)manipulator">
-        <chain base_link="$(arg robot_prefix)base_link" tip_link="$(arg robot_prefix)tool0" />
+    <group name="${robot_prefix}manipulator">
+        <chain base_link="${robot_prefix}base_link" tip_link="${robot_prefix}tool0" />
     </group>
-    <!-- <group name="$(arg robot_prefix)manipulator">
-        <joint name="$(arg robot_prefix)joint_1"/>
-        <joint name="$(arg robot_prefix)joint_2"/>
-        <joint name="$(arg robot_prefix)joint_3"/>
-        <joint name="$(arg robot_prefix)joint_4"/>
-        <joint name="$(arg robot_prefix)joint_5"/>
-        <joint name="$(arg robot_prefix)joint_6"/>
+    <!-- <group name="${robot_prefix}manipulator">
+        <joint name="${robot_prefix}joint_1"/>
+        <joint name="${robot_prefix}joint_2"/>
+        <joint name="${robot_prefix}joint_3"/>
+        <joint name="${robot_prefix}joint_4"/>
+        <joint name="${robot_prefix}joint_5"/>
+        <joint name="${robot_prefix}joint_6"/>
     </group> -->
     <!-- End-Effector -->
-    <group name="$(arg robot_prefix)eoat">
-        <chain base_link="$(arg robot_prefix)base_link" tip_link="$(arg robot_prefix)eoat_tcp" />
+    <group name="${robot_prefix}eoat">
+        <chain base_link="${robot_prefix}base_link" tip_link="${robot_prefix}eoat_tcp" />
     </group>
     <!--GROUP STATES: Purpose: Define a named state for a particular group, in terms of joint values. This is useful to define states like 'folded arms'-->
-    <group_state name="$(arg robot_prefix)init" group="$(arg robot_prefix)manipulator">
-        <joint name="$(arg robot_prefix)joint_1" value="0.000" />
-        <joint name="$(arg robot_prefix)joint_2" value="0.000" />
-        <joint name="$(arg robot_prefix)joint_3" value="0.000" />
-        <joint name="$(arg robot_prefix)joint_4" value="0.000" />
-        <joint name="$(arg robot_prefix)joint_5" value="0.000" />
-        <joint name="$(arg robot_prefix)joint_6" value="0.000" />
+    <group_state name="${robot_prefix}init" group="${robot_prefix}manipulator">
+        <joint name="${robot_prefix}joint_1" value="0.000" />
+        <joint name="${robot_prefix}joint_2" value="0.000" />
+        <joint name="${robot_prefix}joint_3" value="0.000" />
+        <joint name="${robot_prefix}joint_4" value="0.000" />
+        <joint name="${robot_prefix}joint_5" value="0.000" />
+        <joint name="${robot_prefix}joint_6" value="0.000" />
     </group_state>
-    <group_state name="$(arg robot_prefix)home" group="$(arg robot_prefix)manipulator">
-        <joint name="$(arg robot_prefix)joint_1" value="1.5708" />
-        <joint name="$(arg robot_prefix)joint_2" value="-0.720" />
-        <joint name="$(arg robot_prefix)joint_3" value="-0.720" />
-        <joint name="$(arg robot_prefix)joint_4" value="0.000" />
-        <joint name="$(arg robot_prefix)joint_5" value="-1.5708" />
-        <joint name="$(arg robot_prefix)joint_6" value="0.000" />
+    <group_state name="${robot_prefix}home" group="${robot_prefix}manipulator">
+        <joint name="${robot_prefix}joint_1" value="1.5708" />
+        <joint name="${robot_prefix}joint_2" value="-0.720" />
+        <joint name="${robot_prefix}joint_3" value="-0.720" />
+        <joint name="${robot_prefix}joint_4" value="0.000" />
+        <joint name="${robot_prefix}joint_5" value="-1.5708" />
+        <joint name="${robot_prefix}joint_6" value="0.000" />
     </group_state>
     <!--VIRTUAL JOINT: Purpose: this element defines a virtual joint between a robot link and an external frame of reference (considered fixed with respect to the robot)-->
-    <!-- <virtual_joint name="$(arg robot_prefix)world_joint" type="fixed" parent_frame="world" child_link="$(arg robot_prefix)base_link" /> -->
-    <!-- <virtual_joint name="$(arg robot_prefix)link1_adjustment" />
-    <virtual_joint name="$(arg robot_prefix)balancer_A" />
-    <virtual_joint name="$(arg robot_prefix)balancer_B" />
-    <virtual_joint name="$(arg robot_prefix)cylinderbox" /> -->
+    <!-- <virtual_joint name="${robot_prefix}world_joint" type="fixed" parent_frame="world" child_link="${robot_prefix}base_link" /> -->
+    <!-- <virtual_joint name="${robot_prefix}link1_adjustment" />
+    <virtual_joint name="${robot_prefix}balancer_A" />
+    <virtual_joint name="${robot_prefix}balancer_B" />
+    <virtual_joint name="${robot_prefix}cylinderbox" /> -->
     <!--PASSIVE JOINT: Purpose: this element is used to mark joints that are not actuated-->
-    <!-- <passive_joint name="$(arg robot_prefix)link1_adjustment" />
-    <passive_joint name="$(arg robot_prefix)balancer_A" />
-    <passive_joint name="$(arg robot_prefix)balancer_B" />
-    <passive_joint name="$(arg robot_prefix)cylinderbox" /> -->
+    <!-- <passive_joint name="${robot_prefix}link1_adjustment" />
+    <passive_joint name="${robot_prefix}balancer_A" />
+    <passive_joint name="${robot_prefix}balancer_B" />
+    <passive_joint name="${robot_prefix}cylinderbox" /> -->
     <!--DISABLE COLLISIONS: By default it is assumed that any link of the robot could potentially come into collision with any other link in the robot. This tag disables collision checking between a specified pair of links. -->
-    <disable_collisions link1="$(arg robot_prefix)balancer_A" link2="$(arg robot_prefix)balancer_B" reason="Adjacent" />
-    <disable_collisions link1="$(arg robot_prefix)balancer_A" link2="$(arg robot_prefix)cylinderbox" reason="Never" />
-    <disable_collisions link1="$(arg robot_prefix)balancer_A" link2="$(arg robot_prefix)link_1" reason="Default" />
-    <disable_collisions link1="$(arg robot_prefix)balancer_A" link2="$(arg robot_prefix)link_2" reason="Never" />
-    <disable_collisions link1="$(arg robot_prefix)balancer_A" link2="$(arg robot_prefix)link_3" reason="Adjacent" />
-    <disable_collisions link1="$(arg robot_prefix)balancer_A" link2="$(arg robot_prefix)link_4" reason="Never" />
-    <disable_collisions link1="$(arg robot_prefix)balancer_A" link2="$(arg robot_prefix)link_5" reason="Never" />
-    <disable_collisions link1="$(arg robot_prefix)balancer_A" link2="$(arg robot_prefix)link_6" reason="Never" />
-    <disable_collisions link1="$(arg robot_prefix)balancer_B" link2="$(arg robot_prefix)cylinderbox" reason="Never" />
-    <disable_collisions link1="$(arg robot_prefix)balancer_B" link2="$(arg robot_prefix)link_1" reason="Adjacent" />
-    <disable_collisions link1="$(arg robot_prefix)balancer_B" link2="$(arg robot_prefix)link_2" reason="Adjacent" />
-    <disable_collisions link1="$(arg robot_prefix)balancer_B" link2="$(arg robot_prefix)link_3" reason="Never" />
-    <!-- <disable_collisions link1="$(arg robot_prefix)balancer_B" link2="$(arg robot_prefix)link_4" reason="Never" />
-    <disable_collisions link1="$(arg robot_prefix)balancer_B" link2="$(arg robot_prefix)link_5" reason="Never" />
-    <disable_collisions link1="$(arg robot_prefix)balancer_B" link2="$(arg robot_prefix)link_6" reason="Never" /> -->
-    <disable_collisions link1="$(arg robot_prefix)base_link" link2="$(arg robot_prefix)cylinderbox" reason="Never" />
-    <disable_collisions link1="$(arg robot_prefix)base_link" link2="$(arg robot_prefix)link_1" reason="Adjacent" />
-    <disable_collisions link1="$(arg robot_prefix)base_link" link2="$(arg robot_prefix)link_2" reason="Never" />
-    <disable_collisions link1="$(arg robot_prefix)base_link" link2="$(arg robot_prefix)link_3" reason="Never" />
-    <disable_collisions link1="$(arg robot_prefix)base_link" link2="$(arg robot_prefix)link_4" reason="Never" />
-    <disable_collisions link1="$(arg robot_prefix)base_link" link2="$(arg robot_prefix)link_5" reason="Never" />
-    <disable_collisions link1="$(arg robot_prefix)base_link" link2="$(arg robot_prefix)link_6" reason="Never" />
-    <disable_collisions link1="$(arg robot_prefix)cylinderbox" link2="$(arg robot_prefix)link_1" reason="Adjacent" />
-    <disable_collisions link1="$(arg robot_prefix)cylinderbox" link2="$(arg robot_prefix)link_2" reason="Default" />
-    <disable_collisions link1="$(arg robot_prefix)cylinderbox" link2="$(arg robot_prefix)link_4" reason="Never" />
-    <disable_collisions link1="$(arg robot_prefix)cylinderbox" link2="$(arg robot_prefix)link_5" reason="Never" />
-    <disable_collisions link1="$(arg robot_prefix)cylinderbox" link2="$(arg robot_prefix)link_6" reason="Never" />
-    <disable_collisions link1="$(arg robot_prefix)link_1" link2="$(arg robot_prefix)link_2" reason="Adjacent" />
-    <disable_collisions link1="$(arg robot_prefix)link_1" link2="$(arg robot_prefix)link_4" reason="Never" />
-    <disable_collisions link1="$(arg robot_prefix)link_1" link2="$(arg robot_prefix)link_5" reason="Never" />
-    <disable_collisions link1="$(arg robot_prefix)link_1" link2="$(arg robot_prefix)link_6" reason="Never" />
-    <disable_collisions link1="$(arg robot_prefix)link_2" link2="$(arg robot_prefix)link_3" reason="Adjacent" />
-    <disable_collisions link1="$(arg robot_prefix)link_2" link2="$(arg robot_prefix)link_4" reason="Never" />
-    <disable_collisions link1="$(arg robot_prefix)link_2" link2="$(arg robot_prefix)link_5" reason="Never" />
-    <disable_collisions link1="$(arg robot_prefix)link_2" link2="$(arg robot_prefix)link_6" reason="Never" />
-    <disable_collisions link1="$(arg robot_prefix)link_3" link2="$(arg robot_prefix)link_4" reason="Adjacent" />
-    <disable_collisions link1="$(arg robot_prefix)link_3" link2="$(arg robot_prefix)link_5" reason="Never" />
-    <disable_collisions link1="$(arg robot_prefix)link_3" link2="$(arg robot_prefix)link_6" reason="Never" />
-    <disable_collisions link1="$(arg robot_prefix)link_4" link2="$(arg robot_prefix)link_5" reason="Adjacent" />
-    <disable_collisions link1="$(arg robot_prefix)link_4" link2="$(arg robot_prefix)link_6" reason="Never" />
-    <disable_collisions link1="$(arg robot_prefix)link_5" link2="$(arg robot_prefix)link_6" reason="Adjacent" />
+    <disable_collisions link1="${robot_prefix}balancer_A" link2="${robot_prefix}balancer_B" reason="Adjacent" />
+    <disable_collisions link1="${robot_prefix}balancer_A" link2="${robot_prefix}cylinderbox" reason="Never" />
+    <disable_collisions link1="${robot_prefix}balancer_A" link2="${robot_prefix}link_1" reason="Default" />
+    <disable_collisions link1="${robot_prefix}balancer_A" link2="${robot_prefix}link_2" reason="Never" />
+    <disable_collisions link1="${robot_prefix}balancer_A" link2="${robot_prefix}link_3" reason="Adjacent" />
+    <disable_collisions link1="${robot_prefix}balancer_A" link2="${robot_prefix}link_4" reason="Never" />
+    <disable_collisions link1="${robot_prefix}balancer_A" link2="${robot_prefix}link_5" reason="Never" />
+    <disable_collisions link1="${robot_prefix}balancer_A" link2="${robot_prefix}link_6" reason="Never" />
+    <disable_collisions link1="${robot_prefix}balancer_B" link2="${robot_prefix}cylinderbox" reason="Never" />
+    <disable_collisions link1="${robot_prefix}balancer_B" link2="${robot_prefix}link_1" reason="Adjacent" />
+    <disable_collisions link1="${robot_prefix}balancer_B" link2="${robot_prefix}link_2" reason="Adjacent" />
+    <disable_collisions link1="${robot_prefix}balancer_B" link2="${robot_prefix}link_3" reason="Never" />
+    <!-- <disable_collisions link1="${robot_prefix}balancer_B" link2="${robot_prefix}link_4" reason="Never" />
+    <disable_collisions link1="${robot_prefix}balancer_B" link2="${robot_prefix}link_5" reason="Never" />
+    <disable_collisions link1="${robot_prefix}balancer_B" link2="${robot_prefix}link_6" reason="Never" /> -->
+    <disable_collisions link1="${robot_prefix}base_link" link2="${robot_prefix}cylinderbox" reason="Never" />
+    <disable_collisions link1="${robot_prefix}base_link" link2="${robot_prefix}link_1" reason="Adjacent" />
+    <disable_collisions link1="${robot_prefix}base_link" link2="${robot_prefix}link_2" reason="Never" />
+    <disable_collisions link1="${robot_prefix}base_link" link2="${robot_prefix}link_3" reason="Never" />
+    <disable_collisions link1="${robot_prefix}base_link" link2="${robot_prefix}link_4" reason="Never" />
+    <disable_collisions link1="${robot_prefix}base_link" link2="${robot_prefix}link_5" reason="Never" />
+    <disable_collisions link1="${robot_prefix}base_link" link2="${robot_prefix}link_6" reason="Never" />
+    <disable_collisions link1="${robot_prefix}cylinderbox" link2="${robot_prefix}link_1" reason="Adjacent" />
+    <disable_collisions link1="${robot_prefix}cylinderbox" link2="${robot_prefix}link_2" reason="Default" />
+    <disable_collisions link1="${robot_prefix}cylinderbox" link2="${robot_prefix}link_4" reason="Never" />
+    <disable_collisions link1="${robot_prefix}cylinderbox" link2="${robot_prefix}link_5" reason="Never" />
+    <disable_collisions link1="${robot_prefix}cylinderbox" link2="${robot_prefix}link_6" reason="Never" />
+    <disable_collisions link1="${robot_prefix}link_1" link2="${robot_prefix}link_2" reason="Adjacent" />
+    <disable_collisions link1="${robot_prefix}link_1" link2="${robot_prefix}link_4" reason="Never" />
+    <disable_collisions link1="${robot_prefix}link_1" link2="${robot_prefix}link_5" reason="Never" />
+    <disable_collisions link1="${robot_prefix}link_1" link2="${robot_prefix}link_6" reason="Never" />
+    <disable_collisions link1="${robot_prefix}link_2" link2="${robot_prefix}link_3" reason="Adjacent" />
+    <disable_collisions link1="${robot_prefix}link_2" link2="${robot_prefix}link_4" reason="Never" />
+    <disable_collisions link1="${robot_prefix}link_2" link2="${robot_prefix}link_5" reason="Never" />
+    <disable_collisions link1="${robot_prefix}link_2" link2="${robot_prefix}link_6" reason="Never" />
+    <disable_collisions link1="${robot_prefix}link_3" link2="${robot_prefix}link_4" reason="Adjacent" />
+    <disable_collisions link1="${robot_prefix}link_3" link2="${robot_prefix}link_5" reason="Never" />
+    <disable_collisions link1="${robot_prefix}link_3" link2="${robot_prefix}link_6" reason="Never" />
+    <disable_collisions link1="${robot_prefix}link_4" link2="${robot_prefix}link_5" reason="Adjacent" />
+    <disable_collisions link1="${robot_prefix}link_4" link2="${robot_prefix}link_6" reason="Never" />
+    <disable_collisions link1="${robot_prefix}link_5" link2="${robot_prefix}link_6" reason="Adjacent" />
     </xacro:macro>
 </robot>
